File: 120-channel pogo pin board.sch (KiCad schematic (older format))
At the start: 241 parts, among them P1 CONN_1, P10 CONN_1, P100 CONN_1, P101 CONN_1, P102 CONN_1, P103 CONN_1, P104 CONN_1, P105 CONN_1, P106 CONN_1, P107 CONN_1, P108 CONN_1, P109 CONN_1, P11 CONN_1, P110 CONN_1, P111 CONN_1, P112 CONN_1, P113 CONN_1, P114 CONN_1, P115 CONN_1, P116 CONN_1, P117 CONN_1, P118 CONN_1, P119 CONN_1, P12 CONN_1, P120 CONN_1, P121 CONN_1, P13 CONN_1, P14 CONN_1, P15 CONN_1, P16 CONN_1, P17 CONN_1, P18 CONN_1, P19 CONN_1, P2 CONN_1, P20 CONN_1, P21 CONN_1, P22 CONN_1, P23 CONN_1, P24 CONN_1, P25 CONN_1, P26 CONN_1, P27 CONN_1, P28 CONN_1, P29 CONN_1, P3 CONN_1, P30 CONN_1, P31 CONN_1, P32 CONN_1, P33 CONN_1, P34 CONN_1, P35 CONN_1, P36 CONN_1, P37 CONN_1, P38 CONN_1, P39 CONN_1, P4 CONN_1, P40 CONN_1, P41 CONN_1, P42 CONN_1, P43 CONN_1, P44 CONN_1, P45 CONN_1, P46 CONN_1, P47 CONN_1, P48 CONN_1, P49 CONN_1, P5 CONN_1, P50 CONN_1, P51 CONN_1, P52 CONN_1, P53 CONN_1, P54 CONN_1, P55 CONN_1, P56 CONN_1, P57 CONN_1, P58 CONN_1, P59 CONN_1, P6 CONN_1, P60 CONN_1, P61 CONN_1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

Commit message: Update for compatibility with DropBot v3
Parts:
- removed P1, P10, P100, P101, P102, P103, P104, P105, P106, P107, P108, P109, P11, P110, P111, P112, P113, P114, P115, P116, P117, P118, P119, P12, P120, P13, P14, P15, P16, P17, P18, P19, P2, P20, P21, P22, P23, P24, P25, P26, P27, P28, P29, P3, P30, P31, P32, P33, P34, P35, P36, P37, P38, P39, P4, P40, P41, P42, P43, P44, P45, P46, P47, P48, P49, P5, P50, P51, P52, P53, P54, P55, P56, P57, P58, P59, P6, P60, P61, P62, P63, P64, P65, P66, P67, P68, P69, P7, P70, P71, P72, P73, P74, P75, P76, P77, P78, P79, P8, P80, P81, P82, P83, P84, P85, P86, P87, P88, P89, P9, P90, P91, P92, P93, P94, P95, P96, P97, P98, P99: CONN_1, wheelerlab:1.4mm_DMF_Electrode, symbol CONN_1
- removed P121: CONN_1, wheelerlab:3.9mm_DMF_Electrode, symbol CONN_1
- added P1, P10, P100, P101, P102, P103, P104, P105, P106, P107, P108, P109, P11, P110, P111, P112, P113, P114, P115, P116, P117, P118, P119, P12, P120, P122, P123, P124, P125, P126, P127, P128, P129, P13, P130, P131, P132, P133, P134, P135, P136, P137, P14, P15, P16, P17, P18, P19, P2, P20, P21, P22, P23, P24, P25, P26, P27, P28, P29, P3, P30, P31, P32, P33, P34, P35, P36, P37, P38, P39, P4, P40, P41, P42, P43, P44, P45, P46, P47, P48, P49, P5, P50, P51, P52, P53, P54, P55, P56, P57, P58, P59, P6, P60, P61, P62, P63, P64, P65, P66, P67, P68, P69, P7, P70, P71, P72, P73, P74, P75, P76, P77, P78, P79, P8, P80, P81, P82, P83, P84, P85, P86, P87, P88, P89, P9, P90, P91, P92, P93, P94, P95, P96, P97, P98, P99: CONN_01X01, wheelerlab:1.9mm_DMF_Electrode, symbol CONN_01X01
- added P121, P138: CONN_01X01, Pin_Headers:Pin_Header_Straight_1x01_Pitch2.54mm, symbol CONN_01X01
- C1, C10, C100, C101, C102, C103, C104, C105, C106, C107, C108, C109, C11, C110, C111, C112, C113, C114, C115, C116, C117, C118, C119, C12, C120, C13, C14, C15, C16, C17, C18, C19, C2, C20, C21, C22, C23, C24, C25, C26, C27, C28, C29, C3, C30, C31, C32, C33, C34, C35, C36, C37, C38, C39, C4, C40, C41, C42, C43, C44, C45, C46, C47, C48, C49, C5, C50, C51, C52, C53, C54, C55, C56, C57, C58, C59, C6, C60, C61, C62, C63, C64, C65, C66, C67, C68, C69, C7, C70, C71, C72, C73, C74, C75, C76, C77, C78, C79, C8, C80, C81, C82, C83, C84, C85, C86, C87, C88, C89, C9, C90, C91, C92, C93, C94, C95, C96, C97, C98, C99: footprint Capacitors_SMD:C_1206_HandSoldering -> Capacitors_SMD:C_1206
Connections:
- net labels added: CUR_SENSE
- wire segments 6 -> 9
- no-connect marks 0 -> 4
